Commit message: testing and plumbing

File: sphero_rvr_description/urdf/geometry.urdf.xacro (robot description, xacro)
@@ -2,10 +2,12 @@
 <robot xmlns:xacro="http://www.ros.org/wiki/xacro">
 	<!-- robot geometric characteristics -->
-    <xacro:property name="rvr_body_length" value="0.21"/>
-    <xacro:property name="rvr_body_width" value="0.18"/>
-    <xacro:property name="rvr_body_height" value="0.055"/>
-    <xacro:property name="rvr_wheel_width" value="0.05"/>
-    <xacro:property name="rvr_wheel_radius" value="0.07"/>
-    <xacro:property name="rvr_track_length" value="0.19"/>
-    <xacro:property name="rvr_track_link_size" value="0.01"/>
+    <xacro:property name="rvr_body_length" value="0.165"/>
+    <xacro:property name="rvr_body_width" value="0.13"/>
+    <xacro:property name="rvr_body_height" value="0.048"/>
+    <xacro:property name="rvr_wheel_width" value="0.03"/>
+    <xacro:property name="rvr_wheel_diameter" value="0.065"/>
+    <xacro:property name="rvr_wheel_radius" value="${rvr_wheel_diameter/2}"/>
+    <xacro:property name="rvr_track_dz" value="-0.008"/>
+    <xacro:property name="rvr_track_length" value="0.115"/>
+    <xacro:property name="rvr_track_link_size" value="0.002"/>
 </robot>

File: sphero_rvr_description/urdf/materials.urdf.xacro (robot description, xacro)
@@ -33,3 +33,6 @@
     <color rgba="0.8 0.7 0.5 1.0"/>
   </material>
+  <material name="dark_grey">
+    <color rgba="0.2 0.2 0.2 1.0"/>
+  </material>
 </robot>

File: sphero_rvr_description/urdf/wheel.urdf.xacro (robot description, xacro)
@@ -16,5 +16,5 @@
                     <cylinder radius="${rvr_wheel_radius}" length="${rvr_wheel_width}" />
                 </geometry>
-                <material name="LightGrey2"/>
+                <material name="DarkGrey"/>
             </visual>
             <collision >

Commit message: redo urdf geometry

File: sphero_rvr_description/urdf/geometry.urdf.xacro (robot description, xacro)
@@ -2,12 +2,11 @@
 <robot xmlns:xacro="http://www.ros.org/wiki/xacro">
 	<!-- robot geometric characteristics -->
-    <xacro:property name="rvr_body_length" value="0.165"/>
-    <xacro:property name="rvr_body_width" value="0.13"/>
-    <xacro:property name="rvr_body_height" value="0.048"/>
-    <xacro:property name="rvr_wheel_width" value="0.03"/>
+    <xacro:property name="rvr_body_length" value="0.182"/>
+    <xacro:property name="rvr_body_width" value="0.138"/>
+    <xacro:property name="rvr_body_height" value="0.043"/>
+    <xacro:property name="rvr_wheel_width" value="0.035"/>
     <xacro:property name="rvr_wheel_diameter" value="0.065"/>
     <xacro:property name="rvr_wheel_radius" value="${rvr_wheel_diameter/2}"/>
-    <xacro:property name="rvr_track_dz" value="-0.008"/>
-    <xacro:property name="rvr_track_length" value="0.115"/>
-    <xacro:property name="rvr_track_link_size" value="0.002"/>
+    <xacro:property name="rvr_track_dz" value="0.0075"/>
+    <xacro:property name="rvr_track_length" value="${0.062*2}"/>
 </robot>

File: sphero_rvr_description/urdf/sphero_rvr.urdf.xacro (robot description, xacro)
@@ -7,5 +7,5 @@
     <!-- parts -->
     <xacro:include filename="$(find sphero_rvr_description)/urdf/body.urdf.xacro" />
-    <xacro:include filename="$(find sphero_rvr_description)/urdf/track.urdf.xacro" />
+    <xacro:include filename="$(find sphero_rvr_description)/urdf/wheel.urdf.xacro" />
     <!-- urg laser -->
     <xacro:include filename="$(find urg_node)/urdf/hokuyo_ust10.urdf.xacro" />
@@ -15,5 +15,5 @@
     <link name="base_footprint"/>
     <joint name="base_footprint_joint" type="fixed">
-        <origin xyz="0 0 ${-rvr_body_height/2 - 0.01}" rpy="0 0 0" />
+        <origin xyz="0 0 ${rvr_track_dz - rvr_wheel_radius}" rpy="0 0 0" />
         <parent link="base_link" />
         <child link="base_footprint" />
@@ -27,28 +27,19 @@
     <xacro:body name="body" />
     <!-- tracks -->
-    <xacro:track name="left_track" parent="base_link" length="${rvr_track_length}" spin="1" >
-        <origin xyz="0 ${rvr_body_width/2} ${rvr_track_dz}" rpy="0 0 0" />
-    </xacro:track>
-    <xacro:track name="right_track" parent="base_link" length="${rvr_track_length}" spin="-1" >
-        <origin xyz="0 -${rvr_body_width/2} ${rvr_track_dz}" rpy="${M_PI} 0 0" />
-    </xacro:track>
-    <!-- brain -->
-    <link name="pi_sbc" >
-        <origin xyz="0 0 0" rpy="0 0 0" />
-        <visual>
-            <geometry>
-                <box size="0.075 0.055 0.01" />
-            </geometry>
-            <material name="Green"/>
-        </visual>
-    </link>
-    <joint name="pi_sbc_joint" type="fixed" >
-        <parent link="base_link" />
-        <child link="pi_sbc" />
-        <origin xyz="-0.04 0 ${rvr_body_height/2 + 0.012}" rpy="0 0 0" />
-    </joint>
+    <xacro:wheel name="left_track_back_wheel" parent="base_link" direction="1" >
+        <origin xyz="-${rvr_track_length/2} ${rvr_body_width/2} ${rvr_track_dz}" rpy="0 0 0" />
+    </xacro:wheel>
+    <xacro:wheel name="left_track_front_wheel" parent="base_link" direction="1">
+        <origin xyz="${rvr_track_length/2} ${rvr_body_width/2} ${rvr_track_dz}" rpy="0 0 0" />
+    </xacro:wheel>
+    <xacro:wheel name="right_track_back_wheel" parent="base_link" direction="-1" >
+        <origin xyz="-${rvr_track_length/2} -${rvr_body_width/2} ${rvr_track_dz}" rpy="${M_PI} 0 0" />
+    </xacro:wheel>
+    <xacro:wheel name="right_track_front_wheel" parent="base_link" direction="-1">
+        <origin xyz="${rvr_track_length/2} -${rvr_body_width/2} ${rvr_track_dz}" rpy="${M_PI} 0 0" />
+    </xacro:wheel>
     <!-- laser -->
     <xacro:hokuyo_ust10_mount parent_link="base_link" prefix="urg" topic="scan" >
-        <origin xyz="${0.04} 0 ${rvr_body_height/2 + 0.002}" rpy="0 0 0" />
+        <origin xyz="${-0.03} 0 ${rvr_body_height + 0.005}" rpy="0 0 0" />
     </xacro:hokuyo_ust10_mount>
     <!-- gazebo extras -->
