Commit message: setting up gazebo, got model loading and controllers working, wip

File: sphero_rvr_description/urdf/sphero_rvr.urdf.xacro (robot description, xacro)
@@ -37,4 +37,12 @@
             </geometry>
         </collision>
+        <inertial>
+            <origin xyz="0 0 0" rpy="0 0 0"/>
+            <mass value="1.00" />
+            <inertia
+                ixx="${0.001}" ixy="0.0" ixz="0.0"
+                iyy="${0.001}" iyz="0.0"
+                izz="${0.001}"/>
+        </inertial>
     </link>
     <!-- tracks -->
@@ -69,5 +77,4 @@
         <plugin name="gazebo_ros_control" filename="libgazebo_ros_control.so">
             <robotNamespace>/</robotNamespace>
-            <legacyModeNS>true</legacyModeNS>
         </plugin>
     </gazebo>

File: sphero_rvr_description/urdf/track.urdf.xacro (robot description, xacro)
@@ -16,4 +16,12 @@
                 <material name="LightGrey"/>
             </visual>
+            <inertial>
+                <origin xyz="0 0 0" rpy="0 0 0"/>
+                <mass value="0.01" />
+                <inertia
+                    ixx="${0.001}" ixy="0.0" ixz="0.0"
+                    iyy="${0.001}" iyz="0.0"
+                    izz="${0.001}"/>
+            </inertial>
         </link>
         <xacro:wheel name="${name}_back_wheel" parent="${name}" direction="${spin}" >

File: sphero_rvr_description/urdf/wheel.urdf.xacro (robot description, xacro)
@@ -24,4 +24,12 @@
                 </geometry>
             </collision>
+            <inertial>
+                <origin xyz="0 0 0" rpy="0 0 0"/>
+                <mass value="0.076" />
+                <inertia
+                    ixx="${0.001}" ixy="0.0" ixz="0.0"
+                    iyy="${0.001}" iyz="0.0"
+                    izz="${0.001}"/>
+            </inertial>
         </link>
         <gazebo reference="${name}">
@@ -35,5 +43,5 @@
             <type>transmission_interface/SimpleTransmission</type>
             <actuator name="${name}_motor">
-            <mechanicalReduction>1</mechanicalReduction>
+                <mechanicalReduction>1</mechanicalReduction>
             </actuator>
             <joint name="${name}_joint">

Commit message: add mesh model to body

File: sphero_rvr_description/urdf/sphero_rvr.urdf.xacro (robot description, xacro)
@@ -6,4 +6,5 @@
     <xacro:include filename="$(find sphero_rvr_description)/urdf/geometry.urdf.xacro" />
     <!-- parts -->
+    <xacro:include filename="$(find sphero_rvr_description)/urdf/body.urdf.xacro" />
     <xacro:include filename="$(find sphero_rvr_description)/urdf/track.urdf.xacro" />
     <!-- urg laser -->
@@ -24,26 +25,5 @@
     </joint>
     <!-- body acting as base link inertia -->
-    <link name="body" >
-        <origin xyz="0 0 ${rvr_body_height/2}" rpy="0 0 0" />
-        <visual>
-            <geometry>
-                <box size="${rvr_body_length} ${rvr_body_width} ${rvr_body_height}" />
-            </geometry>
-            <material name="White"/>
-        </visual>
-        <collision >
-            <geometry>
-                <box size="${rvr_body_length} ${rvr_body_width} ${rvr_body_height}" />
-            </geometry>
-        </collision>
-        <inertial>
-            <origin xyz="0 0 0" rpy="0 0 0"/>
-            <mass value="1.00" />
-            <inertia
-                ixx="${0.001}" ixy="0.0" ixz="0.0"
-                iyy="${0.001}" iyz="0.0"
-                izz="${0.001}"/>
-        </inertial>
-    </link>
+    <xacro:body name="body" />
     <!-- tracks -->
     <xacro:track name="left_track" parent="base_link" length="${rvr_track_length}" spin="1" >

Commit message: fixes

File: sphero_rvr_description/urdf/sphero_rvr.urdf.xacro (robot description, xacro)
@@ -41,5 +41,5 @@
     <!-- laser -->
     <xacro:hokuyo_ust10_mount parent_link="base_link" prefix="urg" topic="scan" >
-        <origin xyz="${-0.03} 0 ${rvr_body_height + 0.005}" rpy="0 0 0" />
+        <origin xyz="${-0.03} 0 ${rvr_body_height + 0.035}" rpy="0 0 0" />
     </xacro:hokuyo_ust10_mount>
     <!-- gazebo extras -->
