Commit message: testing loc and planning in sim

File: sphero_rvr_description/urdf/body.urdf.xacro (robot description, xacro)
@@ -4,5 +4,4 @@
         <xacro:include filename="$(find sphero_rvr_description)/urdf/geometry.urdf.xacro" />
         <link name="${name}" >
-            <!-- <origin xyz="0 0 ${rvr_body_height/2}" rpy="0 0 0" /> -->
             <visual>
                 <geometry>
@@ -18,9 +17,9 @@
             <inertial>
                 <origin xyz="0 0 0" rpy="0 0 0"/>
-                <mass value="1.00" />
+                <mass value="2.00" />
                 <inertia
-                    ixx="${0.001}" ixy="0.0" ixz="0.0"
-                    iyy="${0.001}" iyz="0.0"
-                    izz="${0.001}"/>
+                    ixx="${0.005}" ixy="0.0" ixz="0.0"
+                    iyy="${0.005}" iyz="0.0"
+                    izz="${0.005}"/>
             </inertial>
         </link>

File: sphero_rvr_description/urdf/wheel.urdf.xacro (robot description, xacro)
@@ -8,5 +8,5 @@
             <xacro:insert_block name="origin" />
             <axis xyz="0 ${direction} 0" rpy="0 0 0" />
-            <limit effort="30" velocity="0.2" />
+            <limit effort="10.0" velocity="50.0" />
         </joint>
         <link name="${name}">
@@ -33,4 +33,17 @@
             </inertial>
         </link>
+        <joint name="${name}_taco_joint" type="fixed">
+            <parent link="${name}" />
+            <child link="${name}_taco" />
+            <origin xyz="0 ${rvr_wheel_width / 2} ${1.05*rvr_wheel_radius}" rpy="0 0 0" />
+        </joint>
+        <link name="${name}_taco">
+            <visual>
+                <geometry>
+                    <cylinder radius="0.005" length="0.004" />
+                </geometry>
+                <material name="Red"/>
+            </visual>
+        </link>
         <gazebo reference="${name}">
 			<mu1 value="1.0"/>
